File: schematic/v1.4/schematic.kicad_pcb (KiCad board)
At the start: 4 copper layers, 85.7 x 22.9 mm, 18 parts, among them J1 USB C 2.0 8Pin, J2 PWR SW, Q1 AO3401, Q2 2N2222, U1 ESP32-C3, U2 4466, U5 WS2812B, U6 AMS1117

Commit message: Final tweaks to pcb
Connections:
- J1 pad A7: Net-(J1-D--PadA7) -> unconnected-(J1-D--PadA7)
Other:
- outline, holes or cut-outs redrawn
Changed lines of the file:
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@@
 			(psnegative no)
 			(psa4output no)
-			(plot_black_and_white yes)
+			(plot_black_and_white no)
 			(sketchpadsonfab no)
 			(plotpadnumbers no)
@@
 			(crossoutdnponfab yes)
 			(subtractmaskfromsilk yes)
-			(outputformat 1)
+			(outputformat 5)
 			(mirror no)
 			(drillshape 0)
@@
 	(net 16 "CC1")
 	(net 17 "unconnected-(J1-SBU1-PadA8)")
-	(net 18 "Net-(J1-D--PadA7)")
+	(net 18 "unconnected-(J1-D--PadA7)")
 	(net 19 "CC2")
 	(net 20 "Net-(Q1-G)")
@@
 	(net 22 "LED D")
 	(net 23 "LED SW")
-	(net 24 "Net-(J2-Pin_1)")
-	(net 25 "unconnected-(U1-D2-Pad6)")
+	(net 24 "unconnected-(U1-D2-Pad6)")
+	(net 25 "Net-(J2-Pin_1)")
 	(footprint "Capacitor_THT:C_Disc_D5.0mm_W2.5mm_P5.00mm"
 		(layer "F.Cu")
@@
 			(remove_unused_layers no)
 			(roundrect_rratio 0.147059)
-			(net 24 "Net-(J2-Pin_1)")
+			(net 25 "Net-(J2-Pin_1)")
 			(pinfunction "Pin_1")
 			(pintype "passive")
@@
 			(layer "F.Fab")
 		)
-		(fp_text user "${REFERENCE}"
-			(at 3.81 0 0)
-			(layer "F.Fab")
-			(effects
-				(font
-					(size 1 1)
-					(thickness 0.15)
-				)
-			)
-		)
 		(pad "1" thru_hole circle
 			(at 0 0)
@@
 			(pinfunction "5V")
 			(pintype "power_in")
-			(thermal_bridge_angle 45)
+			(thermal_bridge_angle 0)
 		)
 		(pad "2" smd roundrect
@@
 			(pinfunction "GND")
 			(pintype "power_in")
-			(thermal_bridge_angle 45)
+			(thermal_bridge_angle 0)
 		)
 		(pad "3" smd roundrect
@@
 			(pinfunction "3V3")
 			(pintype "power_in")
-			(thermal_bridge_angle 45)
+			(thermal_bridge_angle 0)
 		)
 		(pad "4" smd roundrect
@@
 			(pinfunction "D4")
 			(pintype "bidirectional")
-			(thermal_bridge_angle 45)
+			(thermal_bridge_angle 0)
 		)
 		(pad "5" smd roundrect
@@
 			(pinfunction "D3")
 			(pintype "bidirectional")
-			(thermal_bridge_angle 45)
+			(thermal_bridge_angle 0)
 		)
 		(pad "6" smd roundrect
@@
 			(layers "F.Cu" "F.Mask")
 			(roundrect_rratio 0.1388888889)
-			(net 25 "unconnected-(U1-D2-Pad6)")
+			(net 24 "unconnected-(U1-D2-Pad6)")
 			(pinfunction "D2")
 			(pintype "bidirectional+no_connect")
-			(thermal_bridge_angle 45)
+			(thermal_bridge_angle 0)
 		)
 		(pad "7" smd roundrect
@@
 			(pinfunction "D1")
 			(pintype "bidirectional")
-			(thermal_bridge_angle 45)
+			(thermal_bridge_angle 0)
 		)
 		(pad "8" smd roundrect
@@
 			(pinfunction "D0")
 			(pintype "bidirectional")
-			(thermal_bridge_angle 45)
+			(thermal_bridge_angle 0)
 		)
 		(pad "9" smd roundrect
@@
 			(pinfunction "D5")
 			(pintype "bidirectional+no_connect")
-			(thermal_bridge_angle 45)
+			(thermal_bridge_angle 0)
 		)
 		(pad "10" smd roundrect
@@
 			(pinfunction "D6")
 			(pintype "bidirectional")
-			(thermal_bridge_angle 45)
+			(thermal_bridge_angle 0)
 		)
 		(pad "11" smd roundrect
@@
 			(pinfunction "D7")
 			(pintype "bidirectional+no_connect")
-			(thermal_bridge_angle 45)
+			(thermal_bridge_angle 0)
 		)
 		(pad "12" smd roundrect
@@
 			(pinfunction "D8")
 			(pintype "bidirectional+no_connect")
-			(thermal_bridge_angle 45)
+			(thermal_bridge_angle 0)
 		)
 		(pad "13" smd roundrect
@@
 			(pinfunction "D9")
 			(pintype "bidirectional+no_connect")
-			(thermal_bridge_angle 45)
+			(thermal_bridge_angle 0)
 		)
 		(pad "14" smd roundrect
@@
 			(pinfunction "D10")
 			(pintype "bidirectional")
-			(thermal_bridge_angle 45)
+			(thermal_bridge_angle 0)
 		)
 		(pad "15" smd roundrect
@@
 			(pinfunction "D20")
 			(pintype "bidirectional+no_connect")
-			(thermal_bridge_angle 45)
+			(thermal_bridge_angle 0)
 		)
 		(pad "16" smd roundrect
@@
 			(pinfunction "D21")
 			(pintype "bidirectional+no_connect")
-			(thermal_bridge_angle 45)
+			(thermal_bridge_angle 0)
 		)
 		(zone
 			(net 0)
 			(net_name "")
-			(layer "F.SilkS")
+			(layers "F.Cu" "B.Cu")
+			(hatch edge 0.5)
+			(connect_pads
+				(clearance 0)
+			)
+			(min_thickness 0.25)
+			(filled_areas_thickness no)
+			(keepout
+				(tracks not_allowed)
+				(vias not_allowed)
+				(pads not_allowed)
+				(copperpour not_allowed)
+				(footprints not_allowed)
+			)
+			(placement
+				(enabled no)
+				(sheetname "")
+			)
+			(fill
+				(thermal_gap 0.5)
+				(thermal_bridge_width 0.5)
+			)
+			(polygon
+				(pts
+					(xy 77.598081 35.700122) (xy 67.438081 35.700122) (xy 67.438081 31.890122) (xy 77.598081 31.890122)
+				)
+			)
+		)
+		(zone
+			(net 0)
+			(net_name "")
+			(layers "F.Cu" "F.Fab")
 			(hatch edge 0.5)
 			(connect_pads
@@
 				(tracks allowed)
 				(vias allowed)
-				(pads not_allowed)
+				(pads allowed)
 				(copperpour allowed)
 				(footprints not_allowed)
 			)
 			(placement
-				(enabled no)
+				(enabled yes)
 				(sheetname "")
 			)
@@
 			(layers "*.Cu" "*.Mask")
 			(remove_unused_layers no)
-			(net 24 "Net-(J2-Pin_1)")
+			(net 25 "Net-(J2-Pin_1)")
 			(pinfunction "VBUS")
 			(pintype "passive")
@@
 			(layers "*.Cu" "*.Mask")
 			(remove_unused_layers no)
-			(net 18 "Net-(J1-D--PadA7)")
+			(net 18 "unconnected-(J1-D--PadA7)")
 			(pinfunction "D-")
-			(pintype "bidirectional")
+			(pintype "bidirectional+no_connect")
 		)
 		(pad "A8" thru_hole circle
@@
 	)
 	(gr_circle
-		(center 120.75 53.5)
-		(end 120.75 52)
+		(center 120.777 53.467)
+		(end 120.777 51.967)
 		(stroke
 			(width 0.1524)
@@
 	)
 	(segment
-		(start 68.072 35.56)
-		(end 67.931878 35.700122)
-		(width 0.4)
-		(layer "F.Cu")
-		(net 10)
-	)
-	(segment
 		(start 115.25 53.5)
 		(end 114.75 53)
@@
 	(segment
 		(start 69.088 36.576)
-		(end 68.072 35.56)
+		(end 68.58 36.068)
 		(width 0.4)
 		(layer "F.Cu")
@@
 	)
 	(segment
-		(start 67.931878 35.700122)
-		(end 62.993081 35.700122)
+		(start 68.58 36.068)
+		(end 63.360959 36.068)
 		(width 0.4)
 		(layer "F.Cu")
@@
 	)
 	(segment
+		(start 63.360959 36.068)
+		(end 62.993081 35.700122)
+		(width 0.4)
+		(layer "F.Cu")
+		(net 10)
+	)
+	(segment
 		(start 98.206 52.67)
 		(end 98.044 52.832)
@@
 		(width 0.6)
 		(layer "F.Cu")
-		(net 24)
+		(net 25)
 	)
 	(segment
@@
 		(width 0.6)
 		(layer "F.Cu")
-		(net 24)
+		(net 25)
 	)
 	(zone
@@
 		(min_thickness 0.25)
 		(filled_areas_thickness no)
-		(fill yes
+		(fill
 			(thermal_gap 0.5)
 			(thermal_bridge_width 0.5)
@@
 	(group ""
 		(members "38a95f46-e744-4a8c-9cc4-816386a63bd2" "93d1f61c-cf53-4dd6-8fbc-da07353c42db"
-			"97e0dd49-34ee-467c-bee4-a7a138e9c6d9" "cddf7c9d-d36e-41be-b927-ad7d977962f6"
+			"cddf7c9d-d36e-41be-b927-ad7d977962f6"
 		)
 	)

Commit message: Add pcb svg and updates
Parts:
- moved J1 15.7 mm to (32.1, 34.3)
- moved Q2 15.7 mm to (80.8, 42.0)
- moved R4 15.7 mm to (81.8, 34.3)
- moved U5 15.7 mm to (103.7, 24.8)
- moved U6 15.7 mm to (96.0, 38.6)
- moved C5 15.7 mm to (97.5, 34.6)
- moved J2 15.7 mm to (44.0, 26.0)
- moved Q1 15.7 mm to (75.4, 41.6)
- moved R2 15.7 mm to (91.7, 24.9)
- moved U2 15.7 mm to (102.8, 37.8)
- moved C2 15.7 mm to (48.2, 42.7)
- moved U1 15.7 mm to (60.6, 34.4)
- moved C1 15.7 mm to (47.0, 36.6)
- moved C3 15.7 mm to (87.6, 28.5)
- moved C4 15.7 mm to (99.3, 28.3)
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